File: Hardware/BlueSMiRF-ChipAnt.sch (EAGLE design)
At the start: 27 parts, among them Q1 MOSFET-NCHANNELSMD, Q2 MOSFET-NCHANNELSMD, U1 BLUETOOTH-RN41, U3 3.3V

Commit message: Update RES/CAP packages to 0603
Parts:
- C4: device SparkFun:CAP0402-CAP -> SparkFun:CAP0603-CAP
- R1, R2, R3, R4, R5, R6, R7, R8, R9: device SparkFun:RESISTOR0402-RES -> SparkFun:RESISTOR0603-RES

Commit message: Updated board layout
Parts:
- removed JP3: FIDUCIAL1X2, SparkFun:FIDUCIAL1X2

Commit message: Fixing silk screen positions
Parts:
- added U$2: REVISION, SparkFun-Aesthetics:REVISION
Other:
- note added: "J. Lindblom"
- note added: "T. Klopfenstein"
- note removed: "J. Lindblom, T. Klopfenstein"
Changed lines of the file:
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@@
 <part name="TP1" library="SparkFun" deviceset="TEST-POINT" device="3X5" value=""/>
 <part name="LOGO1" library="SparkFun-Aesthetics" deviceset="OSHW-LOGO" device="S"/>
+<part name="U$2" library="SparkFun-Aesthetics" deviceset="REVISION" device=""/>
 </parts>
 <sheets>
@@
 <text x="152.4" y="177.8" size="3.048" layer="97">Level shifting</text>
 <text x="152.4" y="73.66" size="3.048" layer="97">Headers</text>
-<text x="162.56" y="7.62" size="2.54" layer="97">J. Lindblom, T. Klopfenstein</text>
+<text x="171.45" y="11.176" size="2.54" layer="97">J. Lindblom</text>
 <text x="241.3" y="7.62" size="2.54" layer="97">v16</text>
+<text x="174.498" y="6.35" size="2.54" layer="97">T. Klopfenstein</text>
 </plain>
 <instances>
@@
 <instance part="TP1" gate="G$1" x="93.98" y="152.4"/>
 <instance part="LOGO1" gate="G$1" x="134.62" y="10.16"/>
+<instance part="U$2" gate="G$1" x="148.59" y="6.604"/>
 </instances>
 <busses>
